File: Power Sense 3.0/Power Sense 3.0.kicad_pcb (KiCad board)
At the start: 2 copper layers, 133.9 x 50.3 mm, 47 parts, among them IC1 MCP3909, J1 Power, J2 ProgHead, J3 SPI, J4 TestHeader, T1 AC1030, T2 2p2sTransformer, U1 PIC18F25K20_I/SS, Y1 3.579545MHz Crystal

Commit message: Power Sense New Layout
-- Moved Molex connector slot to match up (Not checked very well) to the command board.

-- Need to Still double check the mounting holes!

@Seth let's do a printout again but this time with adopted code
Parts:
- moved REF** 58.2 mm to (74.9, 78.7)
- moved REF** 45.3 mm to (88.4, 57.1)
- moved REF** 43.4 mm to (190.8, 55.9)
- moved J3 24.2 mm to (172.4, 57.8), turned to 0 degrees
- moved J1 8.89 mm to (67.8, 59.5)
- moved R20 8.89 mm to (81.9, 59.6)
- moved R24 8.89 mm to (81.9, 57.0)
- moved C10 6.55 mm to (164.8, 73.9)
- moved U1 5.93 mm to (186.4, 94.5)
- moved D1 4.91 mm to (191.4, 87.1)
- moved D2 4.91 mm to (191.4, 73.7)
- moved D3 4.91 mm to (191.4, 80.4)
- moved R23 4.91 mm to (190.6, 68.2)
- moved R22 4.91 mm to (193.9, 68.2)
- moved R19 4.74 mm to (158.9, 58.5)
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Routing:
- net Net-(C10-Pad1): track 36.0 -> 127.0 mm
- net Net-(R21-Pad2): track 34.6 -> 77.8 mm, vias 0 -> 1
- net GND: track 307.0 -> 280.2 mm, vias 8 -> 9
- net /SPI_MD_IN: track 11.0 -> 34.7 mm
- net /H: track 25.0 -> 43.2 mm
- net /SPI_CLK: track 11.0 -> 28.7 mm
- net /SPI_MD_OUT: track 11.0 -> 28.5 mm
- net Net-(R19-Pad2): track 3.43 -> 20.4 mm
- net Net-(R1-Pad2): track 3.30 -> 16.0 mm
- net /MCLR: track 66.2 -> 78.5 mm, vias 0 -> 1
- net Net-(R18-Pad2): track 29.3 -> 39.9 mm
- net /+5V: track 67.1 -> 76.9 mm
- net Net-(R17-Pad2): track 40.7 -> 49.5 mm
- net /N: track 25.0 -> 16.8 mm
- net /Fo1toPIC: track 84.1 -> 90.7 mm
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Other:
- board text added: "Move Molex Connector UP!"
- board text added: "To CB"
- board text removed: "SPI"
